Commit message: New updated code

File: src/axalta_mir250_robot_ur10e/urdf/axalta_mir250_model_ur10.xacro (robot description, xacro)
@@ -106,5 +106,5 @@
    <parent link="box1" />
    <child link="base_link" />
-     <origin xyz="0 0 0.1217" rpy="0 0 3.1416"/>
+     <origin xyz="0.0 0 0.1217" rpy="0 0 3.1416"/>
    <pose>-0 0 0 0 0 0</pose>
 </joint>
